File: 5hardware/sensor_node_v3/sensor_node.kicad_pcb (KiCad board)
At the start: 2 copper layers, 28 parts, among them J1 Conn_01x03, J3 Conn_01x29, SW2 SW_DIP_x04, SW3 SW_Push, SW4 SW_DIP_x04, SW5 RotaryEncoder, SW6 SW_Push, U1 MCP1700x-330xxTO, U7 CH32V003F4P6, U8 ESP32-WROOM-32D

Commit message: update pcb.
Parts:
- removed SW3: SW_Push, Button_Switch_THT:SW_PUSH_6mm_H7.3mm
- added R13: R, Connector_PinSocket_2.54mm:PinSocket_1x02_P2.54mm_Vertical, F.Cu at (134.3, 39.2)
- added SW1: SW_Push, Button_Switch_THT:SW_PUSH-12mm, F.Cu at (113.3, 107.3)
- SW6: footprint Button_Switch_THT:SW_PUSH-12mm -> Button_Switch_THT:SW_PUSH_6mm_H7.3mm
- U4: moved to F.Cu
- U8: footprint RF_Module:ESP32-WROOM-32D -> A_SensorNode:ESP32-WROOM-32D2
- moved SW6 23.8 mm to (124.2, 128.7), turned to 90 degrees
- moved U8 16.2 mm to (102.7, 139.4)
- moved SW2 1.23 mm to (125.9, 40.6)
- turned U4 to 0 degrees
Connections:
- C2 pad 1: EN -> +3.3V
- J3 pad 1: EN -> +3.3V
- J3 pad 19: AUD (21) -> FREE (21)
- R1 pad 1: EN -> +3.3V
- R10 pad 1: EN -> +3.3V
- R11 pad 2: EN -> +3.3V
- R2 pad 1: EN -> +3.3V
- R3 pad 1: EN -> +3.3V
- R4 pad 1: EN -> +3.3V
- R5 pad 1: EN -> +3.3V
- R7 pad 2: EN -> +3.3V
- R8 pad 1: EN -> +3.3V
- R9 pad 1: EN -> +3.3V
- U1 pad 3: EN -> +3.3V
- U2 pad 19: EN -> +3.3V
- U2 pad 20: EN -> +3.3V
- U2 pad 23: EN -> +3.3V
- U2 pad 24: EN -> +3.3V
- U2 pad 25: EN -> +3.3V
- U2 pad 3: EN -> +3.3V
- U2 pad 31: RX2 (17) -> AUD (17)
- U2 pad 32: TX2 (16) -> Net-(U2-IO_16)
- U2 pad 38: EN -> +3.3V
- U2 pad 4: EN -> +3.3V
- U3 pad 8: EN -> +3.3V
- U4 pad 24: EN -> +3.3V
- U4 pad 3: EN -> +3.3V
- U4 pad 9: EN -> +3.3V
- U5 pad 10: AUD (21) -> AUD (17)
- U5 pad 15: EN -> +3.3V
- U5 pad 19: EN -> +3.3V
- U5 pad 24: EN -> +3.3V
- U5 pad 33: EN -> +3.3V
- U5 pad 37: EN -> +3.3V
- U5 pad 4: EN -> +3.3V
- U5 pad 40: EN -> +3.3V
- U5 pad 44: EN -> +3.3V
- U5 pad 55: EN -> +3.3V
- U5 pad 58: EN -> +3.3V
- U5 pad 61: EN -> +3.3V
- U5 pad 66: EN -> +3.3V
- U5 pad 69: EN -> +3.3V
- U5 pad 7: EN -> +3.3V
- U5 pad 70: EN -> +3.3V
- U5 pad 73: EN -> +3.3V
- U5 pad 76: EN -> +3.3V
- U7 pad 7: EN -> +3.3V
- U8 pad 2: EN -> +3.3V
- U8 pad 33: AUD (21) -> FREE (21)
Routing:
- net +3.3V: track 0.00 -> 412.0 mm, vias 0 -> 4
- net EN: track 390.0 -> 155.0 mm, vias 4 -> 2
- net AUD (21): track 126.9 -> 0.00 mm, vias 4 -> 0
- net Net-(U2-IO_16): track 0.00 -> 97.0 mm, vias 0 -> 1
- net FREE (21): track 0.00 -> 53.4 mm, vias 0 -> 2
- net SCK (18): track 90.5 -> 137.0 mm, vias 2 -> 4
- net IO_36: track 156.9 -> 188.1 mm, vias 4 -> 6
- net GND: track 424.6 -> 455.6 mm, vias 8 -> 10
- net AUD (17): track 0.00 -> 31.0 mm, vias 0 -> 1
- net Net-(U3-RST): track 109.6 -> 134.5 mm, vias 2 -> 5
- net RX2 (17): track 86.9 -> 69.7 mm, vias 3 -> 2
- net Net-(U3-IO_0): track 119.4 -> 106.3 mm
- net SDA1 (2): track 221.0 -> 210.6 mm, vias 5 -> 6
- net IO_34: track 160.6 -> 170.1 mm, vias 3 -> 4
- net MOSI (23): track 137.8 -> 140.1 mm
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Other:
- board outline added: 50.9 x 100.1 mm
- board text added: "0D0"
- board text added: "0D2"
- board text added: "1"
- board text added: "16"
- board text added: "17"
- board text added: "18"
- board text added: "19"
- board text added: "2"
- board text added: "21"
- board text added: "23"
- board text added: "3"
- board text added: "5V"
- board text added: "BLK"
- board text added: "IO0"
- board text added: "LK"
- board text added: "OD0"
- board text added: "OD1"
- board text added: "OD2"
- board text added: "OD3"
- board text added: "OD4"
- board text added: "OD5"
- board text added: "PA1"
- board text added: "PA2"
- board text added: "PC0"
- board text added: "PC4"
- board text added: "PC5"
- board text added: "PC6"
- board text added: "PC7"
- board text added: "PD0"
- board text added: "PD1"
- board text added: "PD2"
- board text added: "PD3"
- board text added: "v+"
- board text added: "x"
- board text removed: "D2"
- board text removed: "DAC"
- board text removed: "IO22"
- board text removed: "MISO"
- board text removed: "MOSI"
- board text removed: "RX2"
- board text removed: "SCK"
- board text removed: "TX2"
- board text removed: "_0"
- board text removed: "_12"
- board text removed: "_13"
- board text removed: "_14"
- board text removed: "_15"
- board text removed: "_16"

Commit message: Complete design phase1.
Other:
- board text added: "ESP-MESS Baseboard V3.0"
Changed lines of the file:
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@@
     (effects (font (size 1 1) (thickness 0.15)) (justify left bottom))
+  )
+  (gr_text "ESP-MESS Baseboard V3.0" (at 107.8 128.6 180) (layer "F.SilkS")
+    (effects (font (size 0.5 0.5) (thickness 0.125)) (justify left bottom))
   )
   (gr_text "12" (at 114.6 114.1) (layer "F.SilkS")
