File: 5hardware/sensor_node_v3/sensor_node.kicad_pcb (KiCad board)
At the start: 2 copper layers, 50.9 x 100.1 mm, 29 parts, among them J1 Conn_01x03, J3 Conn_01x29, SW1 SW_Push, SW2 SW_DIP_x04, SW4 SW_DIP_x04, SW5 RotaryEncoder, SW6 SW_Push, U1 MCP1700x-330xxTO, U7 CH32V003F4P6, U8 ESP32-WROOM-32D

Commit message: update pcb design.
Parts:
- removed R1, R2, R3, R4, R6, R7: R, Connector_PinSocket_2.54mm:PinSocket_1x02_P2.54mm_Vertical
- removed R12: R, Resistor_SMD:R_2512_6332Metric
- R13: footprint Connector_PinSocket_2.54mm:PinSocket_1x02_P2.54mm_Vertical -> Resistor_SMD:R_2512_6332Metric
- U1: moved to B.Cu
- U4: footprint Connector_PinSocket_2.54mm:PinSocket_1x29_P2.54mm_Vertical -> Connector_PinSocket_2.54mm:PinSocket_1x39_P2.54mm_Vertical
- moved J3 71.1 mm to (133.2, 131.2), turned to 180 degrees
- moved U4 71.1 mm to (120.0, 131.2), turned to 180 degrees
- moved U1 44.3 mm to (126.1, 70.5)
- moved R13 43.8 mm to (96.5, 61.5), turned to -90 degrees
- moved R11 10.1 mm to (126.5, 116.6), turned to 90 degrees
- moved R9 8.87 mm to (126.5, 104.5)
- moved R10 7.43 mm to (126.5, 92.5)
- moved R8 4.11 mm to (103.0, 61.5), turned to 90 degrees
- moved SW2 2.85 mm to (128.7, 40.2)
- moved C2 2.45 mm to (126.5, 61.9), turned to -90 degrees
- moved R5 2.31 mm to (109.0, 61.5), turned to 90 degrees
- moved SW6 2.21 mm to (124.3, 130.8)
- moved U7 1.02 mm to (128.0, 52.5), turned to 0 degrees
- turned BZ1 to -90 degrees
- turned SW4 to 90 degrees
Routing:
- net Net-(U3-IO_0): track 106.3 -> 23.1 mm, vias 1 -> 0
- net Net-(U3-D4_SDA): track 98.4 -> 29.0 mm
- net Net-(U3-D5_SCL): track 105.3 -> 35.9 mm
- net OD2: track 57.1 -> 115.4 mm, vias 1 -> 4
- net MOSI (23): track 140.1 -> 197.8 mm, vias 6 -> 5
- net Net-(U3-D3_RX): track 95.3 -> 40.0 mm
- net Net-(J3-Pin_25): track 79.1 -> 24.9 mm, vias 0 -> 1
- net EN: track 155.0 -> 103.6 mm
- net Net-(J3-Pin_24): track 77.7 -> 26.6 mm
- net Net-(J3-Pin_23): track 73.5 -> 24.5 mm, vias 1 -> 0
- net OD1: track 97.3 -> 142.7 mm, vias 4 -> 3
- net Net-(J3-Pin_29): track 105.2 -> 63.7 mm, vias 3 -> 2
- net Net-(U3-D1_TX): track 93.8 -> 54.3 mm
- net IO_36: track 188.1 -> 151.5 mm, vias 6 -> 3
- net SCL (32): track 127.3 -> 163.0 mm, vias 1 -> 2
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Other:
- board text added: "ADC"
- board text added: "D2"
- board text added: "ESP-Mess Baseboard V3.0"
- board text removed: "ESP-MESS Baseboard V3.0"

Commit message: fixing wiring.
Parts:
- added SCL1: TestPoint, TestPoint:TestPoint_Pad_1.5x1.5mm, F.Cu at (92.4, 91.8)
- added SDA1: TestPoint, TestPoint:TestPoint_Pad_1.5x1.5mm, F.Cu at (92.4, 88.2)
- added TP3: TestPoint, TestPoint:TestPoint_Pad_1.5x1.5mm, F.Cu at (135.4, 42.8)
- added TP4: TestPoint, TestPoint:TestPoint_Pad_1.5x1.5mm, F.Cu at (135.0, 47.0)
- added V+: TestPoint, TestPoint:TestPoint_Pad_1.5x1.5mm, F.Cu at (135.6, 130.8)
- added V+: TestPoint, TestPoint:TestPoint_Pad_1.5x1.5mm, F.Cu at (135.6, 38.4)
- added V-: TestPoint, TestPoint:TestPoint_Pad_1.5x1.5mm, F.Cu at (135.6, 127.2)
- added V-: TestPoint, TestPoint:TestPoint_Pad_1.5x1.5mm, F.Cu at (135.6, 34.9)
Routing:
- net SCL (32): track 163.0 -> 114.4 mm
- net SCL1 (0): track 202.5 -> 219.6 mm, vias 5 -> 7
- net +3.3V: track 394.6 -> 409.8 mm, vias 13 -> 14
- net SDA1 (2): track 243.6 -> 255.6 mm, vias 2 -> 4
- net GND: track 461.4 -> 467.7 mm

Commit message: fixing pcb design.
Parts:
- removed SCL1, SDA1, V+ (x2), V- (x2): TestPoint, TestPoint:TestPoint_Pad_1.5x1.5mm
- added TP1: TestPoint, TestPoint:TestPoint_Pad_1.5x1.5mm, F.Cu at (92.2, 152.9)
- added TP2: TestPoint, TestPoint:TestPoint_Pad_1.5x1.5mm, F.Cu at (95.1, 152.9)
- added TP5: TestPoint, TestPoint:TestPoint_Pad_1.5x1.5mm, F.Cu at (134.6, 95.3)
- added TP6: TestPoint, TestPoint:TestPoint_Pad_1.5x1.5mm, F.Cu at (134.6, 98.9)
- added TP7: TestPoint, TestPoint:TestPoint_Pad_1.5x1.5mm, F.Cu at (134.6, 88.0)
- added TP8: TestPoint, TestPoint:TestPoint_Pad_1.5x1.5mm, F.Cu at (134.6, 91.6)
- U1: moved to F.Cu
- moved U3 123.9 mm to (132.4, 153.0), turned to 180 degrees
- moved TP3 115.8 mm to (99.5, 152.9), turned to 180 degrees
- moved TP4 110.8 mm to (102.4, 152.9), turned to 180 degrees
- moved SW2 109.1 mm to (97.3, 144.7), turned to 90 degrees
- moved U8 93.6 mm to (123.5, 48.2), turned to 0 degrees
- moved U7 87.2 mm to (97.2, 134.0)
- moved J3 84.8 mm to (93.5, 56.3), turned to 0 degrees
- moved U4 76.3 mm to (105.8, 56.3), turned to 0 degrees
- moved R13 74.4 mm to (129.7, 128.1), turned to 90 degrees
- moved U2 72.8 mm to (110.2, 102.8)
- moved SW6 71.9 mm to (97.5, 64.1)
- moved R8 69.5 mm to (123.2, 128.0), turned to -90 degrees
- moved C2 69.0 mm to (99.7, 125.4), turned to 90 degrees
- moved R5 67.0 mm to (117.2, 128.0), turned to -90 degrees
- moved R11 50.1 mm to (99.9, 74.1), turned to -90 degrees
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Connections:
- TP3 pad 1: SCL1 (0) -> SCL (32)
- TP4 pad 1: SDA1 (2) -> SDA (33)
- U5 pad 1: SDA1 (2) -> SDA (33)
- U5 pad 12: SCL1 (0) -> SCL (32)
- U5 pad 13: SDA1 (2) -> SDA (33)
- U5 pad 16: SCL1 (0) -> SCL (32)
- U5 pad 17: SDA1 (2) -> SDA (33)
- U5 pad 2: SCL1 (0) -> SCL (32)
- U5 pad 21: SDA1 (2) -> SDA (33)
- U5 pad 22: SCL1 (0) -> SCL (32)
- U5 pad 26: SCL (32) -> SCL1 (0)
- U5 pad 27: SDA (33) -> SDA1 (2)
- U5 pad 30: SDA1 (2) -> SDA (33)
- U5 pad 31: SCL1 (0) -> SCL (32)
- U5 pad 34: SDA (33) -> SDA1 (2)
- U5 pad 35: SCL (32) -> SCL1 (0)
- U5 pad 42: SDA1 (2) -> SDA (33)
- U5 pad 43: SCL1 (0) -> SCL (32)
- U5 pad 52: SDA1 (2) -> SDA (33)
- U5 pad 53: SCL1 (0) -> SCL (32)
- U5 pad 64: SDA1 (2) -> SDA (33)
- U5 pad 65: SCL1 (0) -> SCL (32)
Routing:
- net +3.3V: track 409.8 -> 249.5 mm, vias 14 -> 6
- net SDA1 (2): track 255.6 -> 105.2 mm, vias 4 -> 2
- net MOSI (23): track 197.8 -> 59.0 mm, vias 5 -> 2
- net GND: track 467.7 -> 340.8 mm, vias 7 -> 2
- net SCL1 (0): track 219.6 -> 112.6 mm, vias 7 -> 2
- net SCK (18): track 142.6 -> 54.6 mm, vias 1 -> 0
- net OD5 (15): track 76.8 -> 0.00 mm, vias 2 -> 0
- net MISO (19): track 111.0 -> 35.6 mm, vias 3 -> 1
- net SDA (33): track 115.2 -> 184.8 mm, vias 4 -> 7
- net TX2 (16): track 86.5 -> 18.5 mm, vias 2 -> 1
- net IO_34: track 159.5 -> 92.8 mm, vias 5 -> 4
- net SCL (32): track 114.4 -> 178.1 mm, vias 2 -> 7
- net IO_36: track 151.5 -> 91.6 mm
- net Net-(J3-Pin_27): track 73.1 -> 20.1 mm, vias 4 -> 2
- net OD2: track 115.4 -> 64.5 mm, vias 4 -> 2
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Other:
- board size 50.9 x 100.1 mm -> 49.7 x 100.1 mm

Commit message: updating pcb.
Routing:
- net +3.3V: track 249.5 -> 330.2 mm, vias 6 -> 9
- net AUD (17): track 0.00 -> 80.0 mm, vias 0 -> 1
- net OD5 (15): track 0.00 -> 79.7 mm, vias 0 -> 4
- net SCL (32): track 178.1 -> 244.1 mm, vias 7 -> 9
- net OD4 (13): track 60.3 -> 126.0 mm, vias 1 -> 3
- net GND: track 340.8 -> 401.7 mm, vias 2 -> 4
- net MISO (19): track 35.6 -> 94.2 mm, vias 1 -> 2
- net IO_34: track 92.8 -> 149.9 mm, vias 4 -> 5
- net IO_36: track 91.6 -> 142.8 mm, vias 3 -> 4
- net LLED (4): track 99.4 -> 140.0 mm, vias 2 -> 4
- net MOSI (23): track 59.0 -> 89.4 mm, vias 2 -> 3
- net SCK (18): track 54.6 -> 83.1 mm, vias 0 -> 1
- net BCLK: track 74.3 -> 97.8 mm, vias 1 -> 3
- net OD2: track 64.5 -> 83.7 mm, vias 2 -> 3
- net +5V: track 38.9 -> 41.9 mm, vias 0 -> 1
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
Commit message: fiixing connections.
Parts:
- moved U8 0.17 mm to (123.5, 48.0)
Routing:
- net GND: track 401.7 -> 525.5 mm, vias 4 -> 10
- net +3.3V: track 330.2 -> 428.1 mm, vias 9 -> 16
- net SDA (33): track 184.0 -> 270.7 mm, vias 7 -> 10
- net RST (5): track 96.5 -> 168.4 mm, vias 2 -> 4
- net Net-(J3-Pin_27): track 20.1 -> 90.0 mm, vias 2 -> 4
- net MOSI (23): track 89.4 -> 157.6 mm, vias 3 -> 6
- net OD5 (15): track 79.7 -> 147.3 mm, vias 4 -> 7
- net SCK (18): track 83.1 -> 137.7 mm, vias 1 -> 3
- net Net-(J3-Pin_29): track 13.7 -> 64.6 mm, vias 2 -> 4
- net BCLK: track 97.8 -> 143.6 mm, vias 3 -> 4
- net SCL1 (0): track 112.6 -> 149.8 mm, vias 2 -> 3
- net SDA1 (2): track 105.2 -> 138.2 mm, vias 2 -> 3
- net OD0: track 135.8 -> 162.3 mm, vias 4 -> 5
- net IO_39: track 134.4 -> 159.2 mm, vias 5 -> 8
- net IO_36: track 142.8 -> 166.8 mm, vias 4 -> 6
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