File: 5hardware/sensor_node_v4/sensor_node.kicad_sch (KiCad schematic)
At the start: 39 parts, among them J2 Conn_01x20_Socket, J3 Conn_01x20_Socket, Q2 Si2371EDS, Q3 Si2371EDS, SW3 SW_Push, SW5 SW_Push, SW6 SW_Push, SW7 RotaryEncoder, U1 MCP1700x-330xxTO, U11 MCP1700x-330xxTO, U12 APDS-9960, U14 DS3231M, U15 DS1307+, U16 DS1302+, U17 VL53L1CXV0FY1, U18 BH1750FVI-TR, U4 CH32V003F4P6, U5 SHT31-DIS, U7 XC6206PxxxMR, U8 TPL5110, Y1 Crystal

Commit message: update schematic.
Parts:
- removed BT1: Solar Panel, symbol Device:Battery
- removed U11: MCP1700x-330xxTO, Package_TO_SOT_THT:TO-92_Inline, symbol Regulator_Linear:MCP1700x-330xxTO
- removed U16: DS1302+, Package_DIP:DIP-8_W7.62mm, symbol Timer_RTC:DS1302+
- removed U17: VL53L1CXV0FY1, Sensor_Distance:ST_VL53L1x, symbol Sensor_Distance:VL53L1CXV0FY1
- added BT2: Battery, symbol Device:Battery
- added C3, C4, C5, C6, C7: C, Capacitor_THT:CP_Radial_D5.0mm_P2.00mm, symbol Device:C
- added J1: USB_C_Receptacle_USB2.0, Connector_USB:USB_C_Plug_Molex_105444, symbol Connector:USB_C_Receptacle_USB2.0
- added J4: JYD-41 Connection, symbol Connector:Conn_01x06_Socket
- added P1, P3: S3B-PH-SM4-TB, S3B-PH-SM4-TB:JST_S3B-PH-SM4-TB, symbol JST_S3B-PH:S3B-PH-SM4-TB
- added P2: S4B-PH-SM4-TB, S4B-PH-SM4-TB:JST_S4B-PH-SM4-TB, symbol JST_S4B-PH:S4B-PH-SM4-TB
- added R10, R11, R12, R13, R14, R15, R16, R17, R4, R5, R6, R9: R, Resistor_SMD:R_1206_3216Metric, symbol Device:R
- added R18, R19: R, Resistor_SMD:R_2512_6332Metric, symbol Device:R
- added SW1, SW2: SW_Push, Button_Switch_THT:SW_PUSH-12mm, symbol Switch:SW_Push
- added U2: ~, symbol A_SensorNode:LuatOS_Base2
- D10: footprint (none) -> LED_SMD:LED_1206_3216Metric
- D3, D6: footprint (none) -> LED_SMD:LED_0603_1608Metric
- J2, J3: footprint (none) -> Connector_PinHeader_2.54mm:PinHeader_2x20_P2.54mm_Vertical
- R1: footprint Resistor_SMD:R_2512_6332Metric -> Resistor_SMD:R_1206_3216Metric
- R2, R3, R7, R8: footprint (none) -> Resistor_SMD:R_1206_3216Metric
Connections:
- net D2 is gone; now on net DONE: U9.14 (IO_2)
- net JDY-14 is gone; now on net TX: J2.12 (Pin_12)
- net JDY-7 is gone; now on net JDY-21: J2.7 (Pin_7)
- net JDY-ALED is gone; now on net JDY-18: J2.6 (Pin_6)
- net JDY-RST is gone; now on net JDY-12: J2.4 (Pin_4)
- net JDY-STAT is gone; now on net JDY-PWRC: J2.3 (Pin_3)
- net SCL is gone; now on net SCL (5): J3.15 (Pin_15), J3.19 (Pin_19), J3.8 (Pin_8)
- net SDA is gone; now on net SDA (4): J3.14 (Pin_14), J3.20 (Pin_20), J3.7 (Pin_7)
- net +3.3V: now also U12.5 (LED_A), C3.1, C5.1, C6.1, C7.1, J4.1 (Pin_1), R14.2, R17.2, R9.2, U2.1 (3.3V), U2.15 (3.3V), U2.2 (3.3V), U2.22 (3.3V), U2.30 (3.3V)
- net +5V: now also BT2.1 (+), J1.A4 (VBUS), J1.A9 (VBUS), J1.B4 (VBUS), J1.B9 (VBUS), U2.18 (5V), U2.35 (5V); no longer Q2.2 (S), SW6.1, U8.1 (VDD), U8.6 (EN/ONE_SHOT)
- net D0: now also SW1.2
- net D15: now also R18.1
- net D16: now also R19.1
- net D1_TX: now also J2.16 (Pin_16), P2.3
- net D3_RX: now also J2.17 (Pin_17), P2.4
- net GND: now also J2.11 (Pin_11), J2.15 (Pin_15), R8.2, SW3.1, U14.10 (GND), U14.11 (GND), U14.12 (GND), U14.13 (GND), U14.5 (GND), U14.6 (GND), U14.7 (GND), U14.8 (GND), U14.9 (GND), U5.7 (R), C3.2, C4.2, C5.2, C6.2, C7.2, J1.A1 (GND), J1.A12 (GND), J1.B1 (GND), J1.B12 (GND), J1.S1 (SHIELD), J4.4 (Pin_4), J4.5 (Pin_5), J4.6 (Pin_6), P1.2, P2.2, P3.2, P3.3, R12.2, R13.2, R15.1, R16.1, R18.2, R4.1, SW1.1, SW2.1, U2.16 (GND), U2.19 (GND), U2.20 (GND), U2.21 (GND), U2.29 (GND), U2.3 (GND), U2.36 (GND), U2.9 (GND); no longer R3.1, R8.1, SW3.2
- net JDY-12: now also U6.12 (IO-H); no longer J2.10 (Pin_10)
- net JDY-13: now also J2.5 (Pin_5), U6.13 (IO-I); no longer J2.11 (Pin_11)
- net JDY-18: now also U6.18 (IO-M); no longer J2.13 (Pin_13)
- net JDY-21: now also U6.21 (IO-N); no longer J2.14 (Pin_14)
- net JDY-PWRC: no longer J2.5 (Pin_5)
- net MISO: now also U2.25 (GPIO10)
- net MOSI: now also U2.24 (GPIO3)
- net RST: now also R19.2
- net RX: now also J2.13 (Pin_13), R3.1, J4.3 (Pin_3), U2.5 (GPIO1)
- net SCK: now also U2.23 (GPIO2)
- net SCL (5): now also U2.31 (GPIO5)
- net SDA (4): now also U2.32 (GPIO4)
- net SWIO: now also P1.3
- net TX: now also J4.2 (Pin_2), U2.4 (GPIO0)
- net VCC: now also J2.10 (Pin_10), J2.14 (Pin_14), P1.1, P2.1
- net at Q2.3 (D), U1.3 (VO), U7.3 (VI): now also C4.1, R9.1
- net DONE: now reaches U4.8 (PD0), U8.4 (DONE)
- net D-: now reaches U4.1 (PD4)
- net D-: now also R3.2, SW3.2, J1.A7 (D-), J1.B7 (D-); no longer SW3.1
- net at C2.1, D2.1 (K), U4.6 (PA2): now also R6.2; no longer Q3.2 (S)
- net LUAT_TX: now reaches J2.18 (Pin_18)
- net LUAT_TX: now also U2.11 (TX0)
- net LUAT_RX: now reaches J2.19 (Pin_19)
- net LUAT_RX: now also U2.10 (RX0)
- net at D6.2 (A): now also R11.1; no longer U6.6 (STAT)
- net at U5.2 (ADDR): now also R14.1, R15.2
- net at D3.2 (A): now also R10.2; no longer U6.17 (ALED)
- net at U4.14 (PC4): now also SW2.2; no longer R8.2
- net at SW7.A: now also U4.4 (PD7); no longer U4.20 (PD3)
- net at U18.2 (ADDR): now also R16.2, R17.1
- net at D2.2 (A): now also P3.1
- net at U12.3 (LDR): now also U12.4 (LED_K)
- net at U6.22 (PWRC): now also R8.1
- net JDY-11: no longer names the net of J2.9 (Pin_9)
- net JDY-8: no longer names the net of J2.8 (Pin_8)
- new net: BT2.2 (-), Q2.2 (S), R5.2, SW6.1, U8.1 (VDD)
- new net: J1.A5 (CC1), R13.1
- new net: J1.B5 (CC2), R12.1
- new net: R4.2, R5.1, U8.6 (EN/ONE_SHOT)
- new net: Q3.2 (S), R6.1
- new net: R10.1, U6.17 (ALED)
- new net: R11.2, U6.6 (STAT)
- new net D+: J1.A6 (D+), J1.B6 (D+), U4.20 (PD3)
- no-connect marks 2 -> 4
Other:
- moved on the sheet: BZ2, C2, D10, D2, D3, D6, D8, D9, J2, J3, Q2, Q3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

Commit message: update schematic.
Parts:
- J4: footprint (none) -> Connector_PinHeader_2.00mm:PinHeader_1x06_P2.00mm_Vertical
- P1, P3: footprint S3B-PH-SM4-TB:JST_S3B-PH-SM4-TB -> S3B-PH:JST_S3B-PH-SM4-TB
- P2: footprint S4B-PH-SM4-TB:JST_S4B-PH-SM4-TB -> S4B-PH:JST_S4B-PH-SM4-TB
- RV2: footprint (none) -> EVM3ES:EMV3ESX50B12
- U18: footprint BH1750FVI-TR:XDCR_BH1750FVI-TR -> BH1750:XDCR_BH1750FVI-TR
Changed lines of the file:
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@@
       (effects (font (size 1.27 1.27)) (justify left))
     )
-    (property "Footprint" "S4B-PH-SM4-TB:JST_S4B-PH-SM4-TB" (at 77.47 259.715 0)
+    (property "Footprint" "S4B-PH:JST_S4B-PH-SM4-TB" (at 77.47 259.715 0)
       (effects (font (size 1.27 1.27)) (justify bottom) hide)
     )
@@
       (effects (font (size 1.27 1.27)) (justify left))
     )
-    (property "Footprint" "" (at 43.18 250.19 0)
+    (property "Footprint" "Connector_PinHeader_2.00mm:PinHeader_1x06_P2.00mm_Vertical" (at 43.18 250.19 0)
       (effects (font (size 1.27 1.27)) hide)
     )
@@
       (effects (font (size 1.27 1.27)) (justify left))
     )
-    (property "Footprint" "S3B-PH-SM4-TB:JST_S3B-PH-SM4-TB" (at 77.47 243.84 0)
+    (property "Footprint" "S3B-PH:JST_S3B-PH-SM4-TB" (at 77.47 243.84 0)
       (effects (font (size 1.27 1.27)) (justify bottom) hide)
     )
@@
       (effects (font (size 1.27 1.27)))
     )
-    (property "Footprint" "BH1750FVI-TR:XDCR_BH1750FVI-TR" (at 373.38 61.595 0)
+    (property "Footprint" "BH1750:XDCR_BH1750FVI-TR" (at 373.38 61.595 0)
       (effects (font (size 1.27 1.27)) (justify bottom) hide)
     )
@@
       (effects (font (size 1.27 1.27)) (justify right))
     )
-    (property "Footprint" "" (at 32.385 92.075 0)
+    (property "Footprint" "EVM3ES:EMV3ESX50B12" (at 32.385 92.075 0)
       (effects (font (size 1.27 1.27)) hide)
     )
@@
       (effects (font (size 1.27 1.27)) (justify left))
     )
-    (property "Footprint" "S3B-PH-SM4-TB:JST_S3B-PH-SM4-TB" (at 209.55 48.895 0)
-      (effects (font (size 1.27 1.27)) (justify bottom) hide)
-    )
+    (property "Footprint" "S3B-PH:JST_S3B-PH-SM4-TB" (at 209.55 48.895 0)
+      (effects (font (size 1.27 1.27)) (justify bottom) hide)
+    )
