File: 5hardware/I2C_Base_V0/sensor_node.kicad_pcb (KiCad board)
At the start: 2 copper layers, 58 x 100 mm, 100 parts, among them J1 Conn_01x39_Socket, J2 PJ-320D-A, J3 USB_C_Receptacle_USB2.0, J4 Conn_01x39_Socket, J5 Conn_01x15_Pin, P1 S3B-PH-SM4-TB, P2 S4B-PH-SM4-TB, P3 S3B-PH-SM4-TB, Q1 Si2371EDS, Q2 Si2371EDS, Q3 Si2371EDS, Q5 MMBT5551L, SW1 SW_Push, SW2 RotaryEncoder, SW3 SW_Push, SW4 SW_Push, U10 ESP-12F, U12 APDS-9960, U13 SHT31-DIS, U14 Lolin_Base, U15 DS1307Z+, U16 DS3231M, U17 BH1750FVI-TR, U2 ESP32-C3-WROOM-02, U3 CR2450, U4 CH32V003F4P6, U6 MCP1700x-330xxTO, U7 XC6206PxxxMR, U8 TPL5110, U9 E18-MS1-PCB, Y1 Crystal, Y2 Crystal

Commit message: update PCB.
Parts:
- added J6: Conn_01x07_Pin, Connector_PinSocket_2.00mm:PinSocket_1x07_P2.00mm_Vertical, F.Cu at (164.4, 87.4)
- added R46: R, Resistor_SMD:R_0805_2012Metric, B.Cu at (175.4, 55.1)
- added R47: R, Resistor_SMD:R_0805_2012Metric, B.Cu at (175.4, 47.4)
- added R48: R, Resistor_SMD:R_0805_2012Metric, B.Cu at (175.4, 49.8)
- added R49: R, Resistor_SMD:R_0805_2012Metric, B.Cu at (175.4, 52.7)
- added U11: ~, A_SensorNode:JDY-41, B.Cu at (179.8, 149.9)
- moved R26 0.25 mm to (181.5, 125.5)
Connections:
- J4 pad 34: X -> unconnected-(J4-Pin_34-Pad34)
- U10 pad 15: TX1 -> Net-(U10-RXD)
- U10 pad 16: RX1 -> Net-(U10-TXD)
- U2 pad 11: RX3 -> RX1
- U2 pad 12: TX3 -> TX1
- U2 pad 13: USB- -> unconnected-(U2-GPIO18/USB_D--Pad13)
- U2 pad 14: USB+ -> unconnected-(U2-GPIO19/USB_D+-Pad14)
- U2 pad 17: RX1 -> TX2
- U2 pad 18: TX1 -> RX2
Routing:
- net GND: track 313.5 -> 350.1 mm, vias 33 -> 37
- net TX2: track 0.00 -> 34.7 mm, vias 0 -> 3
- net RX2: track 0.00 -> 22.6 mm, vias 0 -> 1
- net +5V: track 124.2 -> 143.4 mm, vias 7 -> 8
- net TX1: track 174.8 -> 193.8 mm, vias 4 -> 5
- net SCL0: track 272.6 -> 290.2 mm, vias 12 -> 13
- net Net-(U10-RXD): track 0.00 -> 13.6 mm
- net VCC: track 533.4 -> 545.6 mm, vias 15 -> 16
- net Net-(U10-TXD): track 0.00 -> 9.46 mm
- net SDA0: track 281.6 -> 289.8 mm, vias 8 -> 7
- net RX1: track 206.1 -> 211.3 mm, vias 7 -> 9
- net PD2: track 64.4 -> 60.7 mm
- net DO1: track 138.9 -> 142.2 mm
- net Net-(U15-SQW/OUT): track 22.8 -> 20.7 mm
- net Net-(U2-EN/CHIP_PU): track 19.2 -> 20.7 mm
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Other:
- board text added: "5V"
- board text added: "A+"
- board text added: "A-"
- board text added: "ADR"
- board text added: "ANT0"
- board text added: "B.Vi"
- board text added: "B.Vo"
- board text added: "CS0"
- board text added: "CS1"
- board text added: "D15"
- board text added: "D16"
- board text added: "DI0"
- board text added: "DI1"
- board text added: "DI2"
- board text added: "DI3"
- board text added: "DO1"
- board text added: "DO2"
- board text added: "DO3"
- board text added: "DONE"
- board text added: "DRV"
- board text added: "ESP-Mess BaseB V6.0 The Future is Now 01-08-2024"
- board text added: "LED"
- board text added: "MISO"
- board text added: "MOSI"
- board text added: "ROTA"
- board text added: "ROTB"
- board text added: "RST"
- board text added: "RST0"
- board text added: "RX1"
- board text added: "S.Vi"
- board text added: "S.Vo"
- board text added: "SCK"
- board text added: "SCL0"
- board text added: "SCL1"
- board text added: "SDA0"
- board text added: "SDA1"
- board text added: "TX1"
- board text added: "V+"
- board text added: "V-"
- board text added: "Vi+"
- board text added: "Vi-"
- board text added: "Vo"
