File: 5hardware/sensor_node_v11/sensor_node.kicad_pcb (KiCad board)
At the start: 2 copper layers, 23.6 x 48 mm, 42 parts, among them J2 Conn_01x08_Socket, P1 S4B-PH-SM4-TB, Q2 AO3401A, Q3 MMBT5551L, Q4 AO3401A, SW1 SW_Push, SW2 SW_Push, SW3 SW_Push, SW4 SW_Reed, SW5 SW_Push, SW6 SW_Push, U1 ESP-12F, U12 APDS-9960, U13 SHT31-DIS, U17 BH1750FVI-TR, U2 2N7002DW, U3 CR2450, U4 CH32V003F4P6, U7 XC6206PxxxMR, U8 TPL5110

Commit message: update PCB.
Parts:
- moved C6 2.81 mm to (145.6, 72.2)
Routing:
- net V-SENS: track 26.7 -> 25.6 mm
- net SCL: track 59.5 -> 58.6 mm
Other:
- board size 23.6 x 48 mm -> 24.1 x 48 mm
