File: 5hardware/sensor_node_v13/sensor_node.kicad_sch (KiCad schematic)
At the start: 44 parts, among them J2 Conn_01x08_Socket, J3 Conn_01x09_Socket, Q1 AO3400A, Q2 AO3401A, Q4 AO3401A, SW1 SW_Push, SW2 SW_Push, SW3 SW_Push, SW7 SW_Push, U1 ESP-12F, U12 APDS-9960, U13 SHT31-DIS, U17 BH1750FVI-TR, U2 2N7002DW, U3 INA219AxDCN, U7 XC6206PxxxMR, U8 TPL5110

Commit message: update PCB.
Parts:
- removed R18: R, Resistor_SMD:R_0603_1608Metric, symbol Device:R
- removed R19: 0K, Resistor_SMD:R_0402_1005Metric, symbol Device:R
Connections:
- net S1: no longer Q2.3 (D), Q4.3 (D), R12.2, U7.3 (VI)
- new net: Q2.3 (D), Q4.3 (D), R12.2, U7.3 (VI)
Changed lines of the file:
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@@
   (junction (at 314.96 78.105) (diameter 0) (color 0 0 0 0)
   )
-  (junction (at 141.605 57.785) (diameter 0) (color 0 0 0 0)
-  )
   (junction (at 179.705 80.645) (diameter 0) (color 0 0 0 0)
   )
@@
   (junction (at 188.595 92.075) (diameter 0) (color 0 0 0 0)
   )
-  (junction (at 110.49 112.395) (diameter 0) (color 0 0 0 0)
-  )
   (junction (at 354.33 122.555) (diameter 0) (color 0 0 0 0)
-  )
-  (junction (at 110.49 133.985) (diameter 0) (color 0 0 0 0)
   )
   (junction (at 170.18 107.315) (diameter 0) (color 0 0 0 0)
@@
     (stroke (width 0) (type default))
   )
-  (wire (pts (xy 102.235 112.395) (xy 110.49 112.395))
-    (stroke (width 0) (type default))
-  )
   (wire (pts (xy 81.915 97.155) (xy 76.835 97.155))
     (stroke (width 0) (type default))
@@
     (stroke (width 0) (type default))
   )
-  (wire (pts (xy 102.235 121.92) (xy 102.235 124.46))
-    (stroke (width 0) (type default))
-  )
   (wire (pts (xy 354.33 110.49) (xy 343.535 110.49))
     (stroke (width 0) (type default))
@@
     (stroke (width 0) (type default))
   )
-  (wire (pts (xy 102.235 132.08) (xy 102.235 133.985))
-    (stroke (width 0) (type default))
-  )
   (wire (pts (xy 118.745 99.695) (xy 118.745 112.395))
     (stroke (width 0) (type default))
@@
     (stroke (width 0) (type default))
   )
-  (wire (pts (xy 102.235 133.985) (xy 110.49 133.985))
-    (stroke (width 0) (type default))
-  )
   (wire (pts (xy 94.615 76.2) (xy 94.615 80.645))
     (stroke (width 0) (type default) (color 255 0 0 1))
@@
     (stroke (width 0) (type default))
   )
-  (wire (pts (xy 141.605 52.705) (xy 146.685 52.705))
-    (stroke (width 0) (type default))
-  )
   (wire (pts (xy 317.5 80.645) (xy 334.01 80.645))
     (stroke (width 0) (type default))
@@
     (stroke (width 0) (type default))
   )
-  (wire (pts (xy 102.235 114.3) (xy 102.235 112.395))
-    (stroke (width 0) (type default))
-  )
   (wire (pts (xy 113.665 69.215) (xy 113.665 80.645))
     (stroke (width 0) (type default) (color 255 0 0 1))
@@
   )
   (wire (pts (xy 286.385 65.405) (xy 286.385 70.485))
-    (stroke (width 0) (type default))
-  )
-  (wire (pts (xy 141.605 52.705) (xy 141.605 57.785))
     (stroke (width 0) (type default))
   )
@@
     (property "Intersheetrefs" "${INTERSHEET_REFS}" (at 277.7453 100.33 0)
       (effects (font (size 1.27 1.27)) (justify right) hide)
-    )
-  )
-  (global_label "S1" (shape input) (at 146.685 52.705 0) (fields_autoplaced)
-    (effects (font (size 1.27 1.27)) (justify left))
-    (property "Intersheetrefs" "${INTERSHEET_REFS}" (at 152.0892 52.705 0)
-      (effects (font (size 1.27 1.27)) (justify left) hide)
     )
   )
@@
     )
   )
-  (symbol (lib_id "Device:R") (at 102.235 118.11 180) (unit 1)
-    (in_bom yes) (on_board yes) (dnp no)
-    (property "Reference" "R18" (at 102.235 115.57 90)
-      (effects (font (size 1.27 1.27)) (justify left))
-    )
-    (property "Value" "R" (at 102.235 118.745 90)
-      (effects (font (size 1.27 1.27)) (justify left))
-    )
-    (property "Footprint" "Resistor_SMD:R_0603_1608Metric" (at 104.013 118.11 90)
-      (effects (font (size 1.27 1.27)) hide)
-    )
-    (property "Datasheet" "~" (at 102.235 118.11 0)
-      (effects (font (size 1.27 1.27)) hide)
-    )
-    (pin "1")
-    (pin "2")
-    (instances
-      (project "sensor_node"
-        (path "/af3a10dd-48b4-4881-8409-82af1b899ed6"
-          (reference "R18") (unit 1)
-        )
-      )
-    )
-  )
   (symbol (lib_id "power:GND") (at 153.67 187.96 270) (mirror x) (unit 1)
     (in_bom yes) (on_board yes) (dnp no)
@@
         )
       )
-    )
-  )
-  (symbol (lib_id "Device:R") (at 102.235 128.27 180) (unit 1)
-    (in_bom yes) (on_board yes) (dnp no)
-    (property "Reference" "R19" (at 102.235 125.73 90)
-      (effects (font (size 1.27 1.27)) (justify left))
-    )
-    (property "Value" "0K" (at 99.695 127 90)
-      (effects (font (size 1.27 1.27)) (justify left))
-    )
-    (property "Footprint" "Resistor_SMD:R_0402_1005Metric" (at 104.013 128.27 90)
-      (effects (font (size 1.27 1.27)) hide)
-    )
-    (property "Datasheet" "~" (at 102.235 128.27 0)
-      (effects (font (size 1.27 1.27)) hide)
-    )
-    (pin "1")
-    (pin "2")
-    (instances
-      (project "sensor_node"
-        (path "/af3a10dd-48b4-4881-8409-82af1b899ed6"
-          (reference "R19") (unit 1)
-        )
-      )
