File: 5hardware/battery_leds/battery_leds.kicad_sch (KiCad schematic)
At the start: 31 parts, among them J1 Conn_01x03_Pin, Q1 AO3400A, Q2 AO3400A, SW2 SW_Push

Commit message: udpate PCBs.
Other:
- moved on the sheet: J1, SW2
Changed lines of the file:
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@@
   (junction (at 283.845 127) (diameter 0) (color 0 0 255 1)
   )
+  (junction (at 119.38 180.34) (diameter 0) (color 0 0 0 0)
+  )
   (junction (at 238.125 174.625) (diameter 0) (color 255 0 255 1)
   )
@@
   )
   (no_connect (at 189.23 161.29))
+  (no_connect (at 171.45 148.59))
   (no_connect (at 171.45 146.05))
   (no_connect (at 189.23 163.83))
@@
   (no_connect (at 189.23 146.05))
   (no_connect (at 171.45 143.51))
-  (no_connect (at 171.45 148.59))
   (no_connect (at 189.23 158.75))
   (no_connect (at 189.23 148.59))
@@
     (stroke (width 0) (type default))
   )
-  (wire (pts (xy 119.38 158.75) (xy 119.38 166.37))
-    (stroke (width 0) (type default))
-  )
   (wire (pts (xy 159.385 135.255) (xy 159.385 153.67))
     (stroke (width 0) (type default) (color 221 133 0 1))
@@
     (stroke (width 0) (type default) (color 221 133 0 1))
   )
-  (wire (pts (xy 104.14 166.37) (xy 96.52 166.37))
+  (wire (pts (xy 101.6 166.37) (xy 96.52 166.37))
     (stroke (width 0) (type default))
   )
@@
     (stroke (width 0) (type default))
   )
-  (wire (pts (xy 113.03 83.185) (xy 137.16 83.185))
+  (wire (pts (xy 109.22 100.33) (xy 133.35 100.33))
     (stroke (width 0) (type default))
   )
@@
     (stroke (width 0) (type default) (color 255 0 255 1))
   )
-  (wire (pts (xy 128.27 85.725) (xy 137.16 85.725))
+  (wire (pts (xy 124.46 102.87) (xy 133.35 102.87))
     (stroke (width 0) (type default))
   )
@@
     (stroke (width 0) (type default) (color 255 0 255 1))
   )
-  (wire (pts (xy 113.03 83.185) (xy 113.03 78.105))
+  (wire (pts (xy 109.22 100.33) (xy 109.22 95.25))
     (stroke (width 0) (type default))
   )
@@
     (stroke (width 0) (type default) (color 0 0 0 1))
   )
+  (wire (pts (xy 96.52 151.13) (xy 96.52 156.21))
+    (stroke (width 0) (type default))
+  )
   (wire (pts (xy 119.38 166.37) (xy 119.38 169.545))
     (stroke (width 0) (type default))
@@
     (stroke (width 0) (type default) (color 0 0 255 1))
   )
+  (wire (pts (xy 119.38 189.23) (xy 119.38 180.34))
+    (stroke (width 0) (type default))
+  )
   (wire (pts (xy 252.095 104.775) (xy 252.095 99.695))
     (stroke (width 0) (type default))
   )
-  (wire (pts (xy 128.27 80.645) (xy 137.16 80.645))
+  (wire (pts (xy 124.46 97.79) (xy 133.35 97.79))
     (stroke (width 0) (type default))
   )
@@
     (stroke (width 0) (type default) (color 0 0 255 1))
   )
-  (wire (pts (xy 114.3 166.37) (xy 119.38 166.37))
+  (wire (pts (xy 119.38 158.75) (xy 119.38 166.37))
+    (stroke (width 0) (type default))
+  )
+  (wire (pts (xy 111.76 166.37) (xy 119.38 166.37))
     (stroke (width 0) (type default))
   )
@@
     (stroke (width 0) (type default) (color 0 0 0 1))
   )
-  (global_label "SWIO" (shape input) (at 128.27 85.725 180) (fields_autoplaced)
+  (global_label "SWIO" (shape input) (at 124.46 102.87 180) (fields_autoplaced)
     (effects (font (size 1.27 1.27)) (justify right))
-    (property "Intersheetrefs" "${INTERSHEET_REFS}" (at 120.6886 85.725 0)
+    (property "Intersheetrefs" "${INTERSHEET_REFS}" (at 116.8786 102.87 0)
       (effects (font (size 1.27 1.27)) (justify right) hide)
     )
@@
     )
   )
+  (symbol (lib_id "power:PWR_FLAG") (at 96.52 151.13 0) (mirror y) (unit 1)
+    (in_bom yes) (on_board yes) (dnp no)
+    (property "Reference" "#FLG01" (at 96.52 149.225 0)
+      (effects (font (size 1.27 1.27)) hide)
+    )
+    (property "Value" "PWR_FLAG" (at 96.52 146.685 0)
+      (effects (font (size 1.27 1.27)))
+    )
+    (property "Footprint" "" (at 96.52 151.13 0)
+      (effects (font (size 1.27 1.27)) hide)
+    )
+    (property "Datasheet" "~" (at 96.52 151.13 0)
+      (effects (font (size 1.27 1.27)) hide)
+    )
+    (pin "1")
+    (instances
+      (project "battery_leds"
+        (path "/2c34c594-d436-4329-a8f5-990f442bfa53"
+          (reference "#FLG01") (unit 1)
+        )
+      )
+      (project "sensor_node"
+        (path "/af3a10dd-48b4-4881-8409-82af1b899ed6"
+          (reference "#FLG01") (unit 1)
+        )
+      )
+    )
+  )
   (symbol (lib_id "Device:LED") (at 238.125 135.89 90) (unit 1)
     (in_bom yes) (on_board yes) (dnp no)
@@
     )
   )
-  (symbol (lib_id "power:GND") (at 128.27 80.645 270) (mirror x) (unit 1)
-    (in_bom yes) (on_board yes) (dnp no)
-    (property "Reference" "#PWR06" (at 121.92 80.645 0)
-      (effects (font (size 1.27 1.27)) hide)
-    )
-    (property "Value" "GND" (at 123.19 80.645 0)
-      (effects (font (size 1.27 1.27)))
-    )
-    (property "Footprint" "" (at 128.27 80.645 0)
-      (effects (font (size 1.27 1.27)) hide)
-    )
-    (property "Datasheet" "" (at 128.27 80.645 0)
+  (symbol (lib_id "power:GND") (at 124.46 97.79 270) (mirror x) (unit 1)
+    (in_bom yes) (on_board yes) (dnp no)
+    (property "Reference" "#PWR06" (at 118.11 97.79 0)
+      (effects (font (size 1.27 1.27)) hide)
+    )
+    (property "Value" "GND" (at 119.38 97.79 0)
+      (effects (font (size 1.27 1.27)))
+    )
+    (property "Footprint" "" (at 124.46 97.79 0)
+      (effects (font (size 1.27 1.27)) hide)
+    )
+    (property "Datasheet" "" (at 124.46 97.79 0)
       (effects (font (size 1.27 1.27)) hide)
     )
@@
     )
   )
-  (symbol (lib_id "power:+3.3V") (at 113.03 78.105 0) (unit 1)
-    (in_bom yes) (on_board yes) (dnp no)
-    (property "Reference" "#PWR012" (at 113.03 81.915 0)
-      (effects (font (size 1.27 1.27)) hide)
-    )
-    (property "Value" "+3.3V" (at 113.03 74.295 0)
-      (effects (font (size 1.27 1.27)))
-    )
-    (property "Footprint" "" (at 113.03 78.105 0)
-      (effects (font (size 1.27 1.27)) hide)
-    )
-    (property "Datasheet" "" (at 113.03 78.105 0)
+  (symbol (lib_id "power:+3.3V") (at 109.22 95.25 0) (unit 1)
+    (in_bom yes) (on_board yes) (dnp no)
+    (property "Reference" "#PWR012" (at 109.22 99.06 0)
+      (effects (font (size 1.27 1.27)) hide)
+    )
+    (property "Value" "+3.3V" (at 109.22 91.44 0)
+      (effects (font (size 1.27 1.27)))
+    )
+    (property "Footprint" "" (at 109.22 95.25 0)
+      (effects (font (size 1.27 1.27)) hide)
+    )
+    (property "Datasheet" "" (at 109.22 95.25 0)
       (effects (font (size 1.27 1.27)) hide)
     )
@@
     )
   )
-  (symbol (lib_id "Connector:Conn_01x03_Pin") (at 142.24 83.185 0) (mirror y) (unit 1)
+  (symbol (lib_id "Connector:Conn_01x03_Pin") (at 138.43 100.33 0) (mirror y) (unit 1)
     (in_bom yes) (on_board yes) (dnp no) (fields_autoplaced)
-    (property "Reference" "J1" (at 143.51 81.915 0)
+    (property "Reference" "J1" (at 139.7 99.06 0)
       (effects (font (size 1.27 1.27)) (justify right))
     )
-    (property "Value" "Conn_01x03_Pin" (at 143.51 84.455 0)
+    (property "Value" "Conn_01x03_Pin" (at 139.7 101.6 0)
       (effects (font (size 1.27 1.27)) (justify right))
     )
-    (property "Footprint" "Connector_PinHeader_2.00mm:PinHeader_1x03_P2.00mm_Vertical" (at 142.24 83.185 0)
-      (effects (font (size 1.27 1.27)) hide)
-    )
-    (property "Datasheet" "~" (at 142.24 83.185 0)
+    (property "Footprint" "Connector_PinHeader_2.00mm:PinHeader_1x03_P2.00mm_Vertical" (at 138.43 100.33 0)
+      (effects (font (size 1.27 1.27)) hide)
+    )
+    (property "Datasheet" "~" (at 138.43 100.33 0)
       (effects (font (size 1.27 1.27)) hide)
     )
@@
     )
   )
-  (symbol (lib_id "Switch:SW_Push") (at 109.22 166.37 0) (mirror y) (unit 1)
-    (in_bom yes) (on_board yes) (dnp no)
-    (property "Reference" "SW2" (at 102.235 168.91 0)
-      (effects (font (size 1.27 1.27)))
-    )
-    (property "Value" "SW_Push" (at 109.22 168.91 0)
-      (effects (font (size 1.27 1.27)))
-    )
-    (property "Footprint" "Button_Switch_SMD:SW_SPST_PTS810" (at 109.22 161.29 0)
-      (effects (font (size 1.27 1.27)) hide)
-    )
-    (property "Datasheet" "~" (at 109.22 161.29 0)
-      (effects (font (size 1.27 1.27)) hide)
-    )
+  (symbol (lib_id "power:PWR_FLAG") (at 119.38 189.23 0) (mirror x) (unit 1)
+    (in_bom yes) (on_board yes) (dnp no)
+    (property "Reference" "#FLG02" (at 119.38 191.135 0)
+      (effects (font (size 1.27 1.27)) hide)
+    )
+    (property "Value" "PWR_FLAG" (at 119.38 193.675 0)
+      (effects (font (size 1.27 1.27)))
+    )
+    (property "Footprint" "" (at 119.38 189.23 0)
+      (effects (font (size 1.27 1.27)) hide)
+    )
+    (property "Datasheet" "~" (at 119.38 189.23 0)
+      (effects (font (size 1.27 1.27)) hide)
+    )
+    (pin "1")
+    (instances
+      (project "battery_leds"
+        (path "/2c34c594-d436-4329-a8f5-990f442bfa53"
+          (reference "#FLG02") (unit 1)
+        )
+      )
+      (project "sensor_node"
+        (path "/af3a10dd-48b4-4881-8409-82af1b899ed6"
+          (reference "#FLG01") (unit 1)
+        )
+      )
+    )
+  )
+  (symbol (lib_id "Switch:SW_Push") (at 106.68 166.37 0) (mirror y) (unit 1)
+    (in_bom yes) (on_board yes) (dnp no)
+    (property "Reference" "SW2" (at 99.695 168.91 0)
+      (effects (font (size 1.27 1.27)))
+    )
+    (property "Value" "SW_Push" (at 106.68 168.91 0)
+      (effects (font (size 1.27 1.27)))
+    )
+    (property "Footprint" "Button_Switch_SMD:SW_SPST_PTS810" (at 106.68 161.29 0)
+      (effects (font (size 1.27 1.27)) hide)
+    )
+    (property "Datasheet" "~" (at 106.68 161.29 0)
+      (effects (font (size 1.27 1.27)) hide)
+    )
