File: 5hardware/ch32v_board_v1/sensor_node.kicad_pcb (KiCad board)
At the start: 2 copper layers, 24.5 x 32 mm, 20 parts, among them J1 Conn_01x06_Pin, J2 Conn_01x08_Pin, J3 Conn_01x09_Pin, J4 USB_C_Receptacle_USB2.0, J5 Conn_01x09_Pin, SW1 SW_Push, U2 CH32V003F4P6, U3 XC6206PxxxMR

Commit message: udpate PCBs.
Parts:
- removed TP1: TestPoint, A_SensorNode:testpoint
- added PC3: TestPoint, A_SensorNode:testpoint, F.Cu at (156.5, 117.1)
Changed lines of the file:
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@@
       (net 2 "GND") (pinfunction "Pin_6") (pintype "passive") (thermal_bridge_angle 45))
-  )
-  (footprint "A_SensorNode:testpoint" (layer "F.Cu")
-    (at 156.3 117)
-    (property "Sheetfile" "sensor_node.kicad_sch")
-    (property "Sheetname" "")
-    (property "ki_description" "test point")
-    (property "ki_keywords" "test point tp")
-    (attr smd)
-    (fp_text reference "TP1" (at 0 -0.5 unlocked) (layer "F.SilkS")
-        (effects (font (size 1 1) (thickness 0.1)))
-    )
-    (fp_text value "TestPoint" (at 0 1 unlocked) (layer "F.Fab")
-        (effects (font (size 1 1) (thickness 0.15)))
-    )
-    (fp_text user "${REFERENCE}" (at 0 2.5 unlocked) (layer "F.Fab")
-        (effects (font (size 1 1) (thickness 0.15)))
-    )
-    (pad "1" smd roundrect (at 0 0) (size 2 2) (layers "F.Cu" "F.Paste" "F.Mask") (roundrect_rratio 0.25)
-      (net 41 "Net-(U2-PC3)") (pinfunction "1") (pintype "passive"))
   )
   (footprint "A_SensorNode:Jumpper" (layer "F.Cu")
@@
       (rotate (xyz 0 0 0))
     )
+  )
+  (footprint "A_SensorNode:testpoint" (layer "F.Cu")
+    (at 156.5 117.1)
+    (property "Sheetfile" "sensor_node.kicad_sch")
+    (property "Sheetname" "")
+    (property "ki_description" "test point")
+    (property "ki_keywords" "test point tp")
+    (attr smd)
+    (fp_text reference "PC3" (at 0 -0.5 unlocked) (layer "F.SilkS")
+        (effects (font (size 1 1) (thickness 0.1)))
+    )
+    (fp_text value "TestPoint" (at 0 1 unlocked) (layer "F.Fab")
+        (effects (font (size 1 1) (thickness 0.15)))
+    )
+    (fp_text user "${REFERENCE}" (at 0 2.5 unlocked) (layer "F.Fab")
+        (effects (font (size 1 1) (thickness 0.15)))
+    )
+    (pad "1" smd roundrect (at 0 0) (size 2 2) (layers "F.Cu" "F.Paste" "F.Mask") (roundrect_rratio 0.25)
+      (net 41 "Net-(U2-PC3)") (pinfunction "1") (pintype "passive"))
   )
   (footprint "A_SensorNode:Jumpper" (layer "F.Cu")
@@
     (style (thickness 0.15) (arrow_length 1.27) (text_position_mode 0) (extension_height 0.58642) (extension_offset 0.5) keep_text_aligned)
   )
-  (segment (start 159.475 110.575) (end 159.475 116.25) (width 0.25) (layer "F.Cu") (net 1))
+  (segment (start 157.5 118.6) (end 148.3 118.6) (width 0.25) (layer "F.Cu") (net 1))
   (segment (start 158.8 101.8) (end 158.8 106.1) (width 0.25) (layer "F.Cu") (net 1))
-  (segment (start 159.475 116.25) (end 157.125 118.6) (width 0.25) (layer "F.Cu") (net 1))
   (segment (start 152.481017 96.793483) (end 152.3745 96.9) (width 0.25) (layer "F.Cu") (net 1))
   (segment (start 151.799998 93.500001) (end 153.562499 93.5) (width 0.25) (layer "F.Cu") (net 1))
-  (segment (start 159.3 110.4) (end 159.475 110.575) (width 0.25) (layer "F.Cu") (net 1))
+  (segment (start 159.475 110.575) (end 159.475 116.625) (width 0.25) (layer "F.Cu") (net 1))
   (segment (start 148.9 96.9) (end 147.25 95.25) (width 0.25) (layer "F.Cu") (net 1))
   (segment (start 146.507405 93.5) (end 146.9 93.5) (width 0.25) (layer "F.Cu") (net 1))
   (segment (start 146.824999 94.927817) (end 146.824999 93.575001) (width 0.25) (layer "F.Cu") (net 1))
+  (segment (start 159.3 110.4) (end 159.475 110.575) (width 0.25) (layer "F.Cu") (net 1))
+  (segment (start 159.475 116.625) (end 157.5 118.6) (width 0.25) (layer "F.Cu") (net 1))
   (segment (start 148.3 118.6) (end 148.3 117.5) (width 0.25) (layer "F.Cu") (net 1))
   (segment (start 138.545406 118.9) (end 148 118.9) (width 0.25) (layer "F.Cu") (net 1))
@@
   (segment (start 152.481017 96.793483) (end 152.825 97.137466) (width 0.25) (layer "F.Cu") (net 1))
   (segment (start 152.3745 96.9) (end 148.9 96.9) (width 0.25) (layer "F.Cu") (net 1))
-  (segment (start 157.125 118.6) (end 148.3 118.6) (width 0.25) (layer "F.Cu") (net 1))
   (segment (start 148.3 117.5) (end 147.7 116.9) (width 0.25) (layer "F.Cu") (net 1))
   (segment (start 138.145406 119.3) (end 138.545406 118.9) (width 0.25) (layer "F.Cu") (net 1))
