File: 5hardware/esp12_board_v1/sensor_node.kicad_sch (KiCad schematic)
At the start: 14 parts, among them J1 Conn_01x09_Pin, J2 Conn_01x06_Pin, SW2 SW_Push, SW7 SW_Push, U1 ESP-12F

Commit message: update PCBs.
Parts:
- removed D2: LED, LED_SMD:LED_0603_1608Metric, symbol Device:LED
- removed J2: Conn_01x06_Pin, Connector_PinHeader_2.54mm:PinHeader_1x06_P2.54mm_Vertical, symbol Connector:Conn_01x06_Pin
- removed R6: R, Resistor_SMD:R_0603_1608Metric, symbol Device:R
- added C2: 100u, Capacitor_SMD:C_1206_3216Metric, symbol Device:C
- added C4: 10u, Capacitor_SMD:C_0603_1608Metric, symbol Device:C
- added C5: .1u, Capacitor_SMD:C_0603_1608Metric, symbol Device:C
- added J3: Conn_01x09_Pin, Connector_PinHeader_2.54mm:PinHeader_1x09_P2.54mm_Vertical, symbol Connector:Conn_01x09_Pin
- added R3: R, Resistor_SMD:R_0603_1608Metric, symbol Device:R
- C1, C3: value C -> 100u; footprint Capacitor_SMD:C_0603_1608Metric -> Capacitor_SMD:C_1206_3216Metric
- R1: footprint A_SensorNode:Jumpper -> Resistor_SMD:R_0603_1608Metric
Connections:
- net +3.3V: now also C2.1, C4.1, C5.1, J3.1 (Pin_1)
- net EN: now also J3.5 (Pin_5)
- net GND: now also C2.2, C4.2, C5.2, J3.2 (Pin_2), R3.1; no longer R1.2
- net IO16: now also J3.6 (Pin_6)
- net LED2: now also J3.7 (Pin_7)
- net RX: now also J3.4 (Pin_4)
- net SW-A: now also U1.6 (GPIO12); no longer U1.5 (GPIO14)
- net SW-B: now also U1.5 (GPIO14); no longer U1.6 (GPIO12)
- net TX: now also J3.3 (Pin_3)
- net IO0: now reaches SW2.2, U1.12 (GPIO0)
- net IO0: now also J3.8 (Pin_8)
- net ADC: now reaches U1.2 (ADC)
- net ADC: now also R1.1, R3.2
- new net: J3.9 (Pin_9), R1.2
- no-connect marks 8 -> 7
Other:
- moved on the sheet: C1, C3, J1, R10, R13, R2, R4, SW2, SW7, U1

Commit message: udpate PCBs.
Changed lines of the file:
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@@
   (junction (at 212.09 151.765) (diameter 0) (color 0 0 0 0)
   )
+  (junction (at 115.57 114.3) (diameter 0) (color 0 0 0 0)
+  )
   (junction (at 85.725 142.24) (diameter 0) (color 0 0 0 0)
   )
@@
   )
   (junction (at 306.07 177.165) (diameter 0) (color 0 0 0 0)
+  )
+  (junction (at 132.715 104.14) (diameter 0) (color 0 0 0 0)
   )
   (junction (at 134.62 129.54) (diameter 0) (color 0 0 0 0)
@@
     (stroke (width 0) (type default))
   )
-  (wire (pts (xy 137.795 104.14) (xy 128.905 104.14))
+  (wire (pts (xy 137.795 104.14) (xy 132.715 104.14))
     (stroke (width 0) (type default))
   )
@@
     (stroke (width 0) (type default))
   )
+  (wire (pts (xy 125.73 99.06) (xy 125.73 104.14))
+    (stroke (width 0) (type default))
+  )
   (wire (pts (xy 314.96 153.67) (xy 308.61 153.67))
     (stroke (width 0) (type default))
@@
   )
   (wire (pts (xy 97.155 142.24) (xy 107.95 142.24))
+    (stroke (width 0) (type default))
+  )
+  (wire (pts (xy 115.57 109.22) (xy 115.57 114.3))
     (stroke (width 0) (type default))
   )
@@
     (stroke (width 0) (type default))
   )
+  (wire (pts (xy 125.73 104.14) (xy 132.715 104.14))
+    (stroke (width 0) (type default))
+  )
   (wire (pts (xy 107.95 144.78) (xy 107.95 142.24))
     (stroke (width 0) (type default))
@@
     (stroke (width 0) (type default))
   )
-  (wire (pts (xy 128.905 100.965) (xy 128.905 104.14))
+  (wire (pts (xy 132.715 99.06) (xy 132.715 104.14))
     (stroke (width 0) (type default))
   )
@@
     )
   )
+  (symbol (lib_id "power:PWR_FLAG") (at 125.73 99.06 0) (mirror y) (unit 1)
+    (in_bom yes) (on_board yes) (dnp no)
+    (property "Reference" "#FLG01" (at 125.73 97.155 0)
+      (effects (font (size 1.27 1.27)) hide)
+    )
+    (property "Value" "PWR_FLAG" (at 125.73 94.615 0)
+      (effects (font (size 1.27 1.27)))
+    )
+    (property "Footprint" "" (at 125.73 99.06 0)
+      (effects (font (size 1.27 1.27)) hide)
+    )
+    (property "Datasheet" "~" (at 125.73 99.06 0)
+      (effects (font (size 1.27 1.27)) hide)
+    )
+    (pin "1")
+    (instances
+      (project "sensor_node"
+        (path "/af3a10dd-48b4-4881-8409-82af1b899ed6"
+          (reference "#FLG01") (unit 1)
+        )
+      )
+    )
+  )
   (symbol (lib_id "power:+3.3V") (at 307.34 144.145 0) (unit 1)
     (in_bom yes) (on_board yes) (dnp no)
@@
     )
   )
-  (symbol (lib_id "power:+3.3V") (at 128.905 100.965 0) (unit 1)
-    (in_bom yes) (on_board yes) (dnp no)
-    (property "Reference" "#PWR07" (at 128.905 104.775 0)
-      (effects (font (size 1.27 1.27)) hide)
-    )
-    (property "Value" "+3.3V" (at 128.905 97.155 0)
-      (effects (font (size 1.27 1.27)))
-    )
-    (property "Footprint" "" (at 128.905 100.965 0)
-      (effects (font (size 1.27 1.27)) hide)
-    )
-    (property "Datasheet" "" (at 128.905 100.965 0)
-      (effects (font (size 1.27 1.27)) hide)
-    )
+  (symbol (lib_id "power:PWR_FLAG") (at 115.57 109.22 0) (mirror y) (unit 1)
+    (in_bom yes) (on_board yes) (dnp no)
+    (property "Reference" "#FLG02" (at 115.57 107.315 0)
+      (effects (font (size 1.27 1.27)) hide)
+    )
+    (property "Value" "PWR_FLAG" (at 115.57 104.775 0)
+      (effects (font (size 1.27 1.27)))
+    )
+    (property "Footprint" "" (at 115.57 109.22 0)
+      (effects (font (size 1.27 1.27)) hide)
+    )
+    (property "Datasheet" "~" (at 115.57 109.22 0)
+      (effects (font (size 1.27 1.27)) hide)
+    )
+    (pin "1")
+    (instances
+      (project "sensor_node"
+        (path "/af3a10dd-48b4-4881-8409-82af1b899ed6"
+          (reference "#FLG02") (unit 1)
+        )
+      )
+    )
+  )
+  (symbol (lib_id "power:+3.3V") (at 132.715 99.06 0) (unit 1)
+    (in_bom yes) (on_board yes) (dnp no)
+    (property "Reference" "#PWR07" (at 132.715 102.87 0)
+      (effects (font (size 1.27 1.27)) hide)
+    )
+    (property "Value" "+3.3V" (at 132.715 95.25 0)
+      (effects (font (size 1.27 1.27)))
+    )
+    (property "Footprint" "" (at 132.715 99.06 0)
+      (effects (font (size 1.27 1.27)) hide)
+    )
+    (property "Datasheet" "" (at 132.715 99.06 0)
+      (effects (font (size 1.27 1.27)) hide)
+    )
