File: 5hardware/esp32c3_board_v1/sensor_node.kicad_pcb (KiCad board)
At the start: 2 copper layers, 30.1 x 24.7 mm, 25 parts, among them J1 Conn_01x09_Pin, J2 Conn_01x09_Pin, J3 USB_C_Receptacle_USB2.0, Q1 AO3401A, SW1 SW_Push, SW2 SW_Push, U2 ESP32-C3-WROOM-02, U3 XC6206PxxxMR

Commit message: udpate PCBs.
Parts:
- added TP1: TestPoint, A_SensorNode:testpoint, F.Cu at (148.8, 79.7)
Routing:
- net Net-(U3-VI): track 17.6 -> 20.9 mm
Changed lines of the file:
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@@
   (net 26 "IO8")
   (net 27 "IO10")
+  (footprint "A_SensorNode:testpoint" (layer "F.Cu")
+    (at 148.8 79.7)
+    (property "Sheetfile" "sensor_node.kicad_sch")
+    (property "Sheetname" "")
+    (property "ki_description" "test point")
+    (property "ki_keywords" "test point tp")
+    (attr smd)
+    (fp_text reference "TP1" (at 0 -0.5 unlocked) (layer "F.SilkS")
+        (effects (font (size 1 1) (thickness 0.1)))
+    )
+    (fp_text value "TestPoint" (at 0 1 unlocked) (layer "F.Fab")
+        (effects (font (size 1 1) (thickness 0.15)))
+    )
+    (fp_text user "${REFERENCE}" (at 0 2.5 unlocked) (layer "F.Fab")
+        (effects (font (size 1 1) (thickness 0.15)))
+    )
+    (pad "1" smd roundrect (at 0 0) (size 2 2) (layers "F.Cu" "F.Paste" "F.Mask") (roundrect_rratio 0.25)
+      (net 2 "Net-(U3-VI)") (pinfunction "1") (pintype "passive"))
+  )
   (footprint "Capacitor_SMD:C_1206_3216Metric" (layer "F.Cu")
     (at 160.925 71.15)
@@
     (fp_line (start 1.6 0.8) (end -1.6 0.8)
       (stroke (width 0.1) (type solid)) (layer "F.Fab"))
-    (pad "1" smd roundrect (at -1.475 0) (size 1.15 1.8) (layers "F.Cu" "F.Paste" "F.Mask") (roundrect_rratio 0.217391)
+    (pad "1" smd roundrect (at -1.475 0) (size 1.15 1.8) (layers "F.Cu" "F.Paste" "F.Mask") (roundrect_rratio 0.2173913043)
       (net 19 "+3.3V") (pintype "passive"))
-    (pad "2" smd roundrect (at 1.475 0) (size 1.15 1.8) (layers "F.Cu" "F.Paste" "F.Mask") (roundrect_rratio 0.217391)
+    (pad "2" smd roundrect (at 1.475 0) (size 1.15 1.8) (layers "F.Cu" "F.Paste" "F.Mask") (roundrect_rratio 0.2173913043)
       (net 1 "GND") (pintype "passive"))
     (model "${KICAD6_3DMODEL_DIR}/Capacitor_SMD.3dshapes/C_1206_3216Metric.wrl"
@@
     (pad "3" smd roundrect (at 1.1375 0 270) (size 1.325 0.6) (layers "F.Cu" "F.Paste" "F.Mask") (roundrect_rratio 0.25)
       (net 2 "Net-(U3-VI)") (pinfunction "VI") (pintype "power_in"))
-    (model "${KICAD6_3DMODEL_DIR}/Package_TO_SOT_SMD.3dshapes/SOT-23-3.wrl"
+    (model "${KICAD7_3DMODEL_DIR}/Package_TO_SOT_SMD.3dshapes/TSOT-23.step"
       (offset (xyz 0 0 0))
       (scale (xyz 1 1 1))
@@
     (fp_line (start 1.6 0.8) (end -1.6 0.8)
       (stroke (width 0.1) (type solid)) (layer "F.Fab"))
-    (pad "1" smd roundrect (at -1.475 0) (size 1.15 1.8) (layers "F.Cu" "F.Paste" "F.Mask") (roundrect_rratio 0.217391)
+    (pad "1" smd roundrect (at -1.475 0) (size 1.15 1.8) (layers "F.Cu" "F.Paste" "F.Mask") (roundrect_rratio 0.2173913043)
       (net 19 "+3.3V") (pintype "passive"))
-    (pad "2" smd roundrect (at 1.475 0) (size 1.15 1.8) (layers "F.Cu" "F.Paste" "F.Mask") (roundrect_rratio 0.217391)
+    (pad "2" smd roundrect (at 1.475 0) (size 1.15 1.8) (layers "F.Cu" "F.Paste" "F.Mask") (roundrect_rratio 0.2173913043)
       (net 1 "GND") (pintype "passive"))
     (model "${KICAD6_3DMODEL_DIR}/Capacitor_SMD.3dshapes/C_1206_3216Metric.wrl"
@@
     (fp_line (start 1.6 0.8) (end -1.6 0.8)
       (stroke (width 0.1) (type solid)) (layer "F.Fab"))
-    (pad "1" smd roundrect (at -1.475 0) (size 1.15 1.8) (layers "F.Cu" "F.Paste" "F.Mask") (roundrect_rratio 0.217391)
+    (pad "1" smd roundrect (at -1.475 0) (size 1.15 1.8) (layers "F.Cu" "F.Paste" "F.Mask") (roundrect_rratio 0.2173913043)
       (net 19 "+3.3V") (pintype "passive"))
-    (pad "2" smd roundrect (at 1.475 0) (size 1.15 1.8) (layers "F.Cu" "F.Paste" "F.Mask") (roundrect_rratio 0.217391)
+    (pad "2" smd roundrect (at 1.475 0) (size 1.15 1.8) (layers "F.Cu" "F.Paste" "F.Mask") (roundrect_rratio 0.2173913043)
       (net 1 "GND") (pintype "passive"))
     (model "${KICAD6_3DMODEL_DIR}/Capacitor_SMD.3dshapes/C_1206_3216Metric.wrl"
@@
     (style (thickness 0.15) (arrow_length 1.27) (text_position_mode 0) (extension_height 0.58642) (extension_offset 0.5) keep_text_aligned)
   )
+  (segment (start 148.8 78.9) (end 150.4 77.3) (width 0.25) (layer "F.Cu") (net 2))
   (segment (start 147.2 77.3) (end 150.4 77.3) (width 0.25) (layer "F.Cu") (net 2))
   (segment (start 146.125 68.725) (end 146.8 69.4) (width 0.25) (layer "F.Cu") (net 2))
   (segment (start 146.099999 68.024999) (end 146.1 65.7) (width 0.25) (layer "F.Cu") (net 2))
   (segment (start 146.125 68.125) (end 146.125 68.725) (width 0.25) (layer "F.Cu") (net 2))
+  (segment (start 148.8 79.9) (end 148.8 78.9) (width 0.25) (layer "F.Cu") (net 2))
   (via (at 150.4 77.3) (size 0.5) (drill 0.3) (layers "F.Cu" "B.Cu") (net 2))
   (via (at 147.2 77.3) (size 0.5) (drill 0.3) (layers "F.Cu" "B.Cu") (net 2))
