File: 5hardware/esp32c3_board_v1/sensor_node.kicad_sch (KiCad schematic)
At the start: 24 parts, among them J1 Conn_01x09_Pin, J2 Conn_01x09_Pin, J3 USB_C_Receptacle_USB2.0, Q1 AO3401A, SW1 SW_Push, SW2 SW_Push, U2 ESP32-C3-WROOM-02, U3 XC6206PxxxMR

Commit message: udpate PCBs.
Parts:
- added TP1: TestPoint, A_SensorNode:testpoint, symbol Connector:TestPoint
Connections:
- net at C2.1, J3.A4 (VBUS), J3.A9 (VBUS)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: now also TP1.1
Changed lines of the file:
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@@
   (junction (at 112.395 80.645) (diameter 0) (color 0 0 0 0)
+  )
+  (junction (at 122.555 179.705) (diameter 0) (color 0 0 0 0)
   )
   (junction (at 211.455 122.555) (diameter 0) (color 0 0 0 0)
@@
     (stroke (width 0) (type default))
   )
+  (wire (pts (xy 122.555 179.705) (xy 136.525 179.705))
+    (stroke (width 0) (type default))
+  )
   (wire (pts (xy 294.005 102.235) (xy 294.005 86.995))
     (stroke (width 0) (type default))
@@
     (stroke (width 0) (type default))
   )
-  (wire (pts (xy 111.76 179.705) (xy 136.525 179.705))
+  (wire (pts (xy 111.76 179.705) (xy 122.555 179.705))
     (stroke (width 0) (type default))
   )
@@
   )
   (wire (pts (xy 195.58 106.045) (xy 188.595 106.045))
+    (stroke (width 0) (type default))
+  )
+  (wire (pts (xy 122.555 172.085) (xy 122.555 179.705))
     (stroke (width 0) (type default))
   )
@@
         )
       )
+    )
+  )
+  (symbol (lib_id "Connector:TestPoint") (at 122.555 172.085 0) (unit 1)
+    (in_bom yes) (on_board yes) (dnp no) (fields_autoplaced)
+    (property "Reference" "TP1" (at 124.46 167.513 0)
+      (effects (font (size 1.27 1.27)) (justify left))
+    )
+    (property "Value" "TestPoint" (at 124.46 170.053 0)
+      (effects (font (size 1.27 1.27)) (justify left))
+    )
+    (property "Footprint" "A_SensorNode:testpoint" (at 127.635 172.085 0)
+      (effects (font (size 1.27 1.27)) hide)
+    )
+    (property "Datasheet" "~" (at 127.635 172.085 0)
+      (effects (font (size 1.27 1.27)) hide)
+    )
+    (pin "1")
+    (instances
+      (project "sensor_node"
+        (path "/af3a10dd-48b4-4881-8409-82af1b899ed6"
+          (reference "TP1") (unit 1)
+        )
+      )
