File: 5hardware/sensor_board_v1/sensor_node.kicad_pcb (KiCad board)
At the start: 2 copper layers, 24.2 x 24.2 mm, 31 parts, among them J1 Conn_01x09_Pin, Q2 AO3401A, Q3 AO3400A, SW1 SW_Push, SW2 SW_Push, U12 APDS-9960, U13 SHT31-DIS, U17 BH1750FVI-TR, U3 INA219AxDCN, U4 2N7002DW, U7 XC6206PxxxMR, U8 TPL5110

Commit message: update pcb.
Parts:
- moved J1 28.3 mm to (90.3, 86.9), turned to 90 degrees
- moved Q2 27.2 mm to (91.3, 68.5), turned to -90 degrees
- moved R7 26.3 mm to (109.8, 67.9), turned to 180 degrees
- moved R19 26.2 mm to (91.6, 68.9), turned to -90 degrees
- moved R1 22.5 mm to (95.9, 67.9), turned to -90 degrees
- moved R3 22.4 mm to (106.3, 67.9), turned to 0 degrees
- moved Q3 21.1 mm to (91.3, 74.1), turned to -90 degrees
- moved C8 20.7 mm to (92.0, 82.5), turned to 0 degrees
- moved U7 20.0 mm to (91.4, 79.8), turned to 90 degrees
- moved U3 19.4 mm to (100.9, 68.1), turned to 90 degrees
- moved R16 19.2 mm to (92.0, 80.5), turned to 180 degrees
- moved U13 18.4 mm to (108.6, 72.4), turned to 0 degrees
- moved R15 18.4 mm to (100.6, 68.6), turned to 180 degrees
- moved R11 17.7 mm to (108.8, 82.4), turned to 0 degrees
- moved U12 16.7 mm to (108.5, 81.8), turned to 180 degrees
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Other:
- board size 24.2 x 24.2 mm -> 24.2 x 24.3 mm

Commit message: update PCBs.
Parts:
- removed C6: C, Capacitor_SMD:C_0603_1608Metric
- removed R3, R7: R, Resistor_SMD:R_0603_1608Metric
- removed R6: 0K, A_SensorNode:Jumpper
- added R10: 10K, Resistor_SMD:R_0603_1608Metric, F.Cu at (102.0, 73.7)
- added R13: 10K, Resistor_SMD:R_0603_1608Metric, F.Cu at (99.3, 73.7)
- added R4: 0K, A_SensorNode:Jumpper, B.Cu at (102.0, 87.5)
- added R5: R, Resistor_SMD:R_0603_1608Metric, F.Cu at (98.5, 87.9)
- added R9: 0K, A_SensorNode:Jumpper, B.Cu at (103.5, 75.5)
- added U1: SHT4x, Sensor_Humidity:Sensirion_DFN-4_1.5x1.5mm_P0.8mm_SHT4x_NoCentralPad, F.Cu at (94.3, 88.2)
- R15: value R -> 0R
- R2: value R -> 5K
- moved J1 28.6 mm to (112.7, 69.1), turned to -90 degrees
- moved Q2 27.9 mm to (111.8, 87.5), turned to 90 degrees
- moved G*** 27.8 mm to (110.1, 87.2)
- moved R19 26.9 mm to (111.4, 87.1), turned to 90 degrees
- moved R1 23.6 mm to (108.0, 88.1), turned to 90 degrees
- moved Q3 21.8 mm to (111.8, 81.8), turned to 90 degrees
- moved C8 21.1 mm to (111.1, 73.5), turned to 180 degrees
- moved U7 20.7 mm to (111.7, 76.1), turned to -90 degrees
- moved R16 19.8 mm to (111.1, 75.5), turned to 0 degrees
- moved U3 19.7 mm to (102.2, 87.8), turned to -90 degrees
- moved R15 18.8 mm to (102.4, 87.3), turned to 0 degrees
- moved U13 18.1 mm to (94.4, 83.6), turned to 180 degrees
- moved SW1 17.2 mm to (109.3, 81.8), turned to -90 degrees
- moved R11 17.0 mm to (94.3, 73.6), turned to 180 degrees
- moved U12 15.9 mm to (94.6, 74.2), turned to 0 degrees
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Connections:
- C7 pad 1: V-SENS -> /V-SENS
- R2 pad 1: Net-(U17-DVI) -> /V-SENS
- R2 pad 2: V-SENS -> Net-(U17-DVI)
- U12 pad 5: V-SENS -> /V-SENS
- U12 pad 8: V-SENS -> /V-SENS
- U13 pad 2: DONE -> /ADDR
- U13 pad 5: V-SENS -> /V-SENS
- U17 pad 1: V-SENS -> /V-SENS
- U17 pad 2: DONE -> /ADDR
- U3 pad 4: V-SENS -> /V-SENS
- U3 pad 7: DONE -> /ADDR
- U3 pad 8: DONE -> /ADDR
Routing:
- net /V-SENS: track 0.00 -> 62.0 mm, vias 0 -> 6
- net V-SENS: track 56.7 -> 0.00 mm, vias 4 -> 0
- net /ADDR: track 0.00 -> 29.8 mm, vias 0 -> 3
- net DONE: track 55.9 -> 27.2 mm, vias 3 -> 0
- net SCL: track 34.0 -> 46.7 mm
- net SDA: track 50.6 -> 60.6 mm, vias 3 -> 4
- net Vi-: track 45.1 -> 48.3 mm
- net Vi+: track 28.9 -> 31.0 mm
- net Net-(Q2-D): track 17.6 -> 17.0 mm
- net DRIVE: track 16.0 -> 16.6 mm
Other:
- board size 24.2 x 24.3 mm -> 24.7 x 24.6 mm
- board text added: "3.3V"
- board text added: "DONE"
- board text added: "DRV"
- board text added: "GND"
- board text added: "SCL"
- board text added: "SDA"
- board text added: "SWA"
- board text added: "SWB"
- board text added: "Sensor_Base_V1.0 04-01-24"
- board text added: "Vi+"
- board text removed: "ESP-MESS B V13.2"

Commit message: udpate PCBs.
Parts:
- added R3: R, Resistor_SMD:R_0603_1608Metric, F.Cu at (111.7, 82.3)
- C4: value C -> 0.1u
- C7: value C -> 1u
- R15: value 0R -> 0.1R
- R19: moved to F.Cu
- R5: value R -> 10K
- moved Q3 2.40 mm to (111.7, 79.4)
- moved R19 2.35 mm to (111.8, 89.4), turned to 0 degrees
- moved U7 1.81 mm to (111.6, 74.3)
- moved Q2 0.97 mm to (111.8, 86.5)
- moved G*** 0.60 mm to (110.1, 87.8)
Routing:
- net +3.3V: track 14.6 -> 12.0 mm
- net Vi-: track 48.3 -> 49.8 mm
- net Net-(Q2-D): track 17.0 -> 18.2 mm
