File: 5hardware/sensor_board_v1/sensor_node.kicad_sch (KiCad schematic)
At the start: 30 parts, among them J1 Conn_01x09_Pin, Q2 AO3401A, Q3 AO3400A, SW1 SW_Push, SW2 SW_Push, U12 APDS-9960, U13 SHT31-DIS, U17 BH1750FVI-TR, U3 INA219AxDCN, U4 2N7002DW, U7 XC6206PxxxMR, U8 TPL5110

Commit message: update pcb.
Parts:
- added R4: 0K, A_SensorNode:Jumpper, symbol Device:R
Connections:
- net Vi+: now also R4.2
- net Vi-: now also R4.1
Other:
- moved on the sheet: R15
Changed lines of the file:
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@@
   (junction (at 322.58 146.05) (diameter 0) (color 0 0 0 0)
   )
-  (junction (at 278.13 142.875) (diameter 0) (color 0 0 0 0)
+  (junction (at 271.145 142.875) (diameter 0) (color 0 0 0 0)
   )
   (junction (at 266.7 90.17) (diameter 0) (color 0 0 0 0)
@@
   (junction (at 174.625 113.665) (diameter 0) (color 0 0 0 0)
   )
-  (junction (at 278.13 154.94) (diameter 0) (color 0 0 0 0)
+  (junction (at 278.765 154.94) (diameter 0) (color 0 0 0 0)
+  )
+  (junction (at 278.765 142.875) (diameter 0) (color 0 0 0 0)
+  )
+  (junction (at 271.145 154.94) (diameter 0) (color 0 0 0 0)
   )
   (junction (at 133.985 103.505) (diameter 0) (color 0 0 0 0)
@@
     (stroke (width 0) (type default))
   )
+  (wire (pts (xy 278.765 153.035) (xy 278.765 154.94))
+    (stroke (width 0) (type default))
+  )
   (wire (pts (xy 93.98 198.755) (xy 99.695 198.755))
     (stroke (width 0) (type default) (color 255 0 0 1))
@@
     (stroke (width 0) (type default))
   )
+  (wire (pts (xy 278.765 142.875) (xy 285.75 142.875))
+    (stroke (width 0) (type default))
+  )
   (wire (pts (xy 281.94 113.665) (xy 283.845 113.665))
     (stroke (width 0) (type default))
@@
     (stroke (width 0) (type default))
   )
+  (wire (pts (xy 278.765 154.94) (xy 285.75 154.94))
+    (stroke (width 0) (type default))
+  )
   (wire (pts (xy 139.065 111.125) (xy 133.985 111.125))
     (stroke (width 0) (type default))
@@
     (stroke (width 0) (type default))
   )
-  (wire (pts (xy 272.415 154.94) (xy 278.13 154.94))
+  (wire (pts (xy 265.43 154.94) (xy 271.145 154.94))
     (stroke (width 0) (type default) (color 255 0 0 1))
   )
@@
     (stroke (width 0) (type default))
   )
-  (wire (pts (xy 272.415 142.875) (xy 278.13 142.875))
+  (wire (pts (xy 265.43 142.875) (xy 271.145 142.875))
     (stroke (width 0) (type default) (color 255 0 0 1))
   )
@@
     (stroke (width 0) (type default))
   )
+  (wire (pts (xy 278.765 142.875) (xy 278.765 145.415))
+    (stroke (width 0) (type default))
+  )
   (wire (pts (xy 276.225 98.425) (xy 276.225 111.125))
     (stroke (width 0) (type default))
@@
     (stroke (width 0) (type default))
   )
-  (wire (pts (xy 278.13 142.875) (xy 285.75 142.875))
+  (wire (pts (xy 271.145 142.875) (xy 278.765 142.875))
     (stroke (width 0) (type default))
   )
@@
     (stroke (width 0) (type default))
   )
-  (wire (pts (xy 278.13 153.035) (xy 278.13 154.94))
+  (wire (pts (xy 271.145 153.035) (xy 271.145 154.94))
     (stroke (width 0) (type default))
   )
@@
     (stroke (width 0) (type default))
   )
-  (wire (pts (xy 278.13 154.94) (xy 285.75 154.94))
+  (wire (pts (xy 271.145 154.94) (xy 278.765 154.94))
     (stroke (width 0) (type default))
   )
@@
     (stroke (width 0) (type default))
   )
-  (wire (pts (xy 278.13 145.415) (xy 278.13 142.875))
+  (wire (pts (xy 271.145 145.415) (xy 271.145 142.875))
     (stroke (width 0) (type default))
   )
@@
     )
   )
-  (global_label "Vi+" (shape input) (at 272.415 142.875 180) (fields_autoplaced)
+  (global_label "Vi+" (shape input) (at 265.43 142.875 180) (fields_autoplaced)
     (effects (font (size 1.27 1.27)) (justify right))
-    (property "Intersheetrefs" "${INTERSHEET_REFS}" (at 266.164 142.875 0)
+    (property "Intersheetrefs" "${INTERSHEET_REFS}" (at 259.179 142.875 0)
       (effects (font (size 1.27 1.27)) (justify right) hide)
     )
@@
     )
   )
-  (global_label "Vi-" (shape input) (at 272.415 154.94 180) (fields_autoplaced)
+  (global_label "Vi-" (shape input) (at 265.43 154.94 180) (fields_autoplaced)
     (effects (font (size 1.27 1.27)) (justify right))
-    (property "Intersheetrefs" "${INTERSHEET_REFS}" (at 266.164 154.94 0)
+    (property "Intersheetrefs" "${INTERSHEET_REFS}" (at 259.179 154.94 0)
       (effects (font (size 1.27 1.27)) (justify right) hide)
     )
@@
         (path "/af3a10dd-48b4-4881-8409-82af1b899ed6"
           (reference "R1") (unit 1)
+        )
+      )
+    )
+  )
+  (symbol (lib_id "Device:R") (at 278.765 149.225 180) (unit 1)
+    (in_bom yes) (on_board yes) (dnp no)
+    (property "Reference" "R4" (at 278.765 146.685 90)
+      (effects (font (size 1.27 1.27)) (justify left))
+    )
+    (property "Value" "0K" (at 276.225 147.955 90)
+      (effects (font (size 1.27 1.27)) (justify left))
+    )
+    (property "Footprint" "A_SensorNode:Jumpper" (at 280.543 149.225 90)
+      (effects (font (size 1.27 1.27)) hide)
+    )
+    (property "Datasheet" "~" (at 278.765 149.225 0)
+      (effects (font (size 1.27 1.27)) hide)
+    )
+    (pin "1")
+    (pin "2")
+    (instances
+      (project "sensor_node"
+        (path "/af3a10dd-48b4-4881-8409-82af1b899ed6"
+          (reference "R4") (unit 1)
         )
       )
@@
     )
   )
-  (symbol (lib_id "Device:R") (at 278.13 149.225 180) (unit 1)
-    (in_bom yes) (on_board yes) (dnp no)
-    (property "Reference" "R15" (at 278.13 146.685 90)
-      (effects (font (size 1.27 1.27)) (justify left))
-    )
-    (property "Value" "R" (at 278.13 149.86 90)
-      (effects (font (size 1.27 1.27)) (justify left))
-    )
-    (property "Footprint" "Resistor_SMD:R_2512_6332Metric" (at 279.908 149.225 90)
-      (effects (font (size 1.27 1.27)) hide)
-    )
-    (property "Datasheet" "~" (at 278.13 149.225 0)
-      (effects (font (size 1.27 1.27)) hide)
-    )
+  (symbol (lib_id "Device:R") (at 271.145 149.225 180) (unit 1)
+    (in_bom yes) (on_board yes) (dnp no)
+    (property "Reference" "R15" (at 271.145 146.685 90)
+      (effects (font (size 1.27 1.27)) (justify left))
+    )
+    (property "Value" "R" (at 271.145 149.86 90)
+      (effects (font (size 1.27 1.27)) (justify left))
+    )
+    (property "Footprint" "Resistor_SMD:R_2512_6332Metric" (at 272.923 149.225 90)
+      (effects (font (size 1.27 1.27)) hide)
+    )
+    (property "Datasheet" "~" (at 271.145 149.225 0)
+      (effects (font (size 1.27 1.27)) hide)
+    )

Commit message: update PCBs.
Parts:
- removed C6: C, Capacitor_SMD:C_0603_1608Metric, symbol Device:C
- removed R3, R7: R, Resistor_SMD:R_0603_1608Metric, symbol Device:R
- removed R6: 0K, A_SensorNode:Jumpper, symbol Device:R
- added R10, R13: 10K, Resistor_SMD:R_0603_1608Metric, symbol Device:R
- added R5: R, Resistor_SMD:R_0603_1608Metric, symbol Device:R
- added R9: 0K, A_SensorNode:Jumpper, symbol Device:R
- added U1: SHT4x, Sensor_Humidity:Sensirion_DFN-4_1.5x1.5mm_P0.8mm_SHT4x_NoCentralPad, symbol Sensor_Humidity:SHT4x
- R15: value R -> 0R
- R2: value R -> 5K
Connections:
- net +3.3V: now also R9.2
- net DONE: no longer U13.2 (ADDR), U17.2 (ADDR), U3.7 (A0), U3.8 (A1)
- net GND: now also R5.1, U1.4 (VSS)
- net SCL: now also R13.1, U1.2 (SCL)
- net SDA: now also R10.1, U1.1 (SDA)
- net V-SENS: now also R2.1, R10.2, R13.2, R9.1, U1.3 (VDD); no longer R2.2
- net at C4.1, U17.5 (DVI): now also R2.2; no longer R2.1
- new net ADDR: R5.2, U13.2 (ADDR), U17.2 (ADDR), U3.7 (A0), U3.8 (A1)
Other:
- moved on the sheet: C4, C7, C8, J1, Q2, Q3, R1, R11, R12, R15, R16, R17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

Commit message: udpate PCBs.
Parts:
- added R3: R, Resistor_SMD:R_0603_1608Metric, symbol Device:R
- C4: value C -> 0.1u
- C7: value C -> 1u
- R15: value 0R -> 0.1R
- R5: value R -> 10K
Connections:
- net DRIVE: now also R3.2
- net GND: now also R3.1
Other:
- moved on the sheet: C4, C7, R1, R12, R2, U12, U17, U7
